File: DCJ11CoreBoard.kicad_pcb (KiCad board)
At the start: 4 copper layers, 160 x 110 mm, 199 parts, among them J1 Conn_01x30_Pin, J2 Conn_01x30_Pin, Q1 SS8050, Q10 SS8050, Q11 SS8050, Q12 SS8050, Q13 SS8050, Q14 SS8050, Q15 SS8050, Q16 SS8050, Q17 SS8050, Q18 SS8050, Q19 SS8050, Q2 SS8050, Q20 SS8050, Q3 SS8050, Q4 SS8050, Q5 SS8050, Q6 SS8050, Q7 SS8050, Q8 SS8050, Q9 SS8050, U1 TPS54302, U10 SN74CB3T3245PWR, U11 SN74CB3T3245PWR, U12 TPRT9193-12GB, U13 SY8089AAAC, U14 SD-CARD_11P, U15 P25Q32SH-SSH-IT, U16 CH347T, U2 CH221K, U3 CY62167EV30LL-45ZXI, U4 CY62167EV30LL-45ZXI, U5 SN74CB3T3245PWR, U6 SN74CB3T3245PWR, U7 GW1N-LV9LQ144C6_I5, U8 DCJ11, U9 SN74CB3T3245PWR, X1 9BC18000151060C3, X2 X50328MSB2GI

Commit message: update hardware design rev 1.1
Parts:
- removed LED7: SZYY0603B1, JLCImport:SZYY0603B1
- added LED27: SZYY0603B1, JLCImport:SZYY0603B1, F.Cu at (100.0, 33.1)
- added R67: 1kΩ, PCM_JLCPCB:R_0603, B.Cu at (161.7, 114.4)
- turned C43 to 180 degrees
Connections:
- C1 pad 2: VCC -> Net-(U2-VDD)
- R3 pad 2: VCC -> Net-(U2-VDD)
- U14 pad 3: +3V3 -> GND
- U14 pad 4: GND -> +3V3
- U2 pad 1: VCC -> Net-(U2-VDD)
Routing:
- net Net-(U2-VDD): track 0.00 -> 4.66 mm
- net VCC: track 3.36 -> 1.21 mm
- added copper zone on B.Cu, net GND
Other:
- board text added: "DCJ-11 Core Board rev 1.1 CYP2D6 6/2/2026"
- board text removed: "DCJ-11 Core Board CYP2D6 5/23/2026"
