File: DCJ11CoreBoard.kicad_sch (KiCad schematic)
At the start: 197 parts, among them J1 Conn_01x30_Pin, J2 Conn_01x30_Pin, Q1 SS8050, Q10 SS8050, Q11 SS8050, Q12 SS8050, Q13 SS8050, Q14 SS8050, Q15 SS8050, Q16 SS8050, Q17 SS8050, Q18 SS8050, Q19 SS8050, Q2 SS8050, Q20 SS8050, Q3 SS8050, Q4 SS8050, Q5 SS8050, Q6 SS8050, Q7 SS8050, Q8 SS8050, Q9 SS8050, U1 TPS54302, U10 SN74CB3T3245PWR, U11 SN74CB3T3245PWR, U12 TPRT9193-12GB, U13 SY8089AAAC, U14 SD-CARD_11P, U15 P25Q32SH-SSH-IT, U16 CH347T, U2 CH221K, U3 CY62167EV30LL-45ZXI, U4 CY62167EV30LL-45ZXI, U5 SN74CB3T3245PWR, U6 SN74CB3T3245PWR, U7 GW1N-LV9LQ144C6_I5, U8 DCJ11, U9 SN74CB3T3245PWR, X1 9BC18000151060C3, X2 X50328MSB2GI

Commit message: update hardware design rev 1.1
Parts:
- removed LED7: SZYY0603B1, JLCImport:SZYY0603B1, symbol JLCImport:SZYY0603B1
- added LED27: SZYY0603B1, JLCImport:SZYY0603B1, symbol JLCImport:SZYY0603B1
- added R67: 1kΩ, PCM_JLCPCB:R_0603, symbol PCM_JLCPCB-Resistors:0603,1kΩ
Connections:
- net +3V3: now also U14.4 (VDD); no longer U14.3 (VSS1)
- net GND: now also U14.3 (VSS1); no longer U14.4 (VDD)
- net VCC: now also R67.1; no longer C1.2, R3.2, U2.1 (VDD)
- net at R47.2: now also LED27.1 (A)
- net at Q1.3 (C): now also LED27.2 (C)
- new net: C1.2, R3.2, R67.2, U2.1 (VDD)
