File: DCJ11CoreBoard_v1.2.kicad_pcb (KiCad board)
At the start: 6 copper layers, 180 x 120 mm, 202 parts, among them Q1 BSS138W, Q2 BSS84, Q3 BSS138W, U1 DCJ11, U10 SY8089AAAC, U11 SN74CB3T3245PWR, U12 SN74CB3T3245PWR, U13 SN74CB3T3245PWR, U14 ME6211A12M3G-N, U15 ME6211A25M3G-N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

Commit message: modify the value of PD negotiation chip's cfg resistor
Parts:
- removed R4: 4.7kΩ, PCM_JLCPCB:R_0603
- added R52: 47kΩ, PCM_JLCPCB:R_0402, B.Cu at (183.2, 120.4)
Other:
- board text added: "DCJ-11 Core Board CYP2D6 rev 1.2 6/24/2026"
- board text removed: "DCJ-11 Core Board CYP2D6 rev 1.2 6/12/2026"
